Commit message: Direction of knees are changed

File: rsc/urdf/tekir3mesh_new_V2.urdf (robot description, URDF)
Before this commit: robot tekirV3, 17 links, 16 joints
Joints:
- joint footFrame_lb: origin xyz=0 0 -0.224282 rpy=0 -0.52359877559 0 -> xyz=0 0 -0.224282 rpy=0 0.52359877559 0
- joint footFrame_rb: origin xyz=0 0 -0.224282 rpy=0 -0.52359877559 0 -> xyz=0 0 -0.224282 rpy=0 0.52359877559 0
