Commit message: last updates

File: rsc/urdf/tekir3mesh.urdf (robot description, URDF)
Before this commit: robot tekirV2, 33 links, 32 joints
Joints:
- joint footLinkFrame_lb: origin xyz=0 0 -0.224282 rpy=0 -0.52359877559 0 -> xyz=0 0 -0.224282 rpy=0 0.52359877559 0
- joint footLinkFrame_rb: origin xyz=0 0 -0.224282 rpy=0 -0.52359877559 0 -> xyz=0 0 -0.224282 rpy=0 0.52359877559 0
